File: eagle/houston.sch (EAGLE design)
At the start: 80 parts, among them Q1 2N3906, Q2 2N3906, Q3 2N3906, Q4 2N3906, Q5 2N3906, Q6 2N3906, Q7 2N3906, Q8 2N3906, U1 TLC5940-NT, U2 TLC5940-NT, X2 HD44780LCD-1602

Commit message: Updating schematic files and source code
Parts:
- C5: value 470uF -> 1000uF
Connections:
- removed net N$122: LED1.A6, Q8.C
- removed net N$123: LED1.A4, Q6.C
- removed net N$124: LED1.A2, Q3.C
- removed net N$125: LED1.A0, Q5.C
- new net N$38: LED1.CB0, U1.OUT15
- new net N$39: LED1.CB1, U1.OUT14
- new net N$42: LED1.CB2, U1.OUT13
- new net N$43: LED1.CB3, U1.OUT12
- net N$47: now also LED1.CB4, U1.OUT11; no longer LED1.CB0, U1.OUT0
- net N$48: now also LED1.CB5, U1.OUT10; no longer LED1.CB1, U1.OUT1
- net N$49: now also LED1.CB6, U1.OUT9; no longer LED1.CB2, U1.OUT2
- net N$50: now also LED1.CB7, U1.OUT8; no longer LED1.CB4, U1.OUT4
- net N$51: now also LED1.CR0, U1.OUT7; no longer LED1.CB3, U1.OUT3
- net N$52: now also LED1.CR1, U1.OUT6; no longer LED1.CB5, U1.OUT5
- net N$53: now also LED1.CR2, U1.OUT5; no longer LED1.CB6, U1.OUT6
- net N$54: now also LED1.CR3, U1.OUT4; no longer LED1.CB7, U1.OUT7
- net N$55: now also LED1.CR4, U1.OUT3; no longer LED1.CR0, U1.OUT8
- net N$56: now also LED1.CR5, U1.OUT2; no longer LED1.CR1, U1.OUT9
- net N$57: now also LED1.CR6, U1.OUT1; no longer LED1.CR2, U1.OUT10
- net N$58: now also LED1.CR7, U1.OUT0; no longer LED1.CR3, U1.OUT11
- net N$59: now also LED1.A4, Q2.C; no longer LED1.CR4, U1.OUT12
- net N$60: now also LED1.A2, Q4.C; no longer LED1.CR5, U1.OUT13
- net N$61: now also LED1.A0, Q7.C; no longer LED1.CR6, U1.OUT14
- net N$62: now also LED1.A6, Q1.C; no longer LED1.CR7, U1.OUT15
- net N$87: now also LED1.A1, Q8.C; no longer LED1.A3, Q2.C
- net N$92: now also LED1.A3, Q6.C; no longer LED1.A5, Q4.C
- net N$93: now also LED1.A5, Q3.C; no longer LED1.A1, Q1.C
- net N$99: now also Q5.C; no longer Q7.C
